Commit message: dog project milestone 1

File: body.urdf (robot description, URDF)
Before this commit: robot robot, 9 links, 8 joints
Links:
- added link GrabberCenter, mass 1; collision box size=0.1 1 0.1; visual box size=0.1 1 0.1
- added link GrabberLeft, mass 1; collision box size=1 0.1 0.1; visual box size=1 0.1 0.1
- added link GrabberRight, mass 1; collision box size=1 0.1 0.1; visual box size=1 0.1 0.1
- added link NeckArm, mass 1; collision box size=1 0.1 0.1; visual box size=1 0.1 0.1
- added link NeckBase, mass 1; collision box size=0.1 0.1 1; visual box size=0.1 0.1 1
- link BackLeg: geometry collision box size=1 0.2 0.2; visual box size=1 0.2 0.2
- link FrontLeg: geometry collision box size=1 0.2 0.2; visual box size=1 0.2 0.2
- link Torso: geometry collision box size=2 1 0.5; visual box size=2 1 0.5
Joints:
- added joint GrabberCenter_GrabberLeft: type revolute, parent GrabberCenter, child GrabberLeft, origin xyz=0 0.5 0 rpy=0 0 0, axis 0 0 1, limit lower=-3.14159 upper=3.14159 effort=0.0 velocity=0.0
- added joint GrabberCenter_GrabberRight: type revolute, parent GrabberCenter, child GrabberRight, origin xyz=0 -0.5 0 rpy=0 0 0, axis 0 0 1, limit lower=-3.14159 upper=3.14159 effort=0.0 velocity=0.0
- added joint NeckArm_GrabberCenter: type revolute, parent NeckArm, child GrabberCenter, origin xyz=1 0 0 rpy=0 0 0, axis 0 1 0, limit lower=-3.14159 upper=3.14159 effort=0.0 velocity=0.0
- added joint NeckBase_NeckArm: type revolute, parent NeckBase, child NeckArm, origin xyz=0 0 1 rpy=0 0 0, axis 1 1 0, limit lower=-3.14159 upper=3.14159 effort=0.0 velocity=0.0
- added joint Torso_NeckBase: type revolute, parent Torso, child NeckBase, origin xyz=0.75 0 1 rpy=0 0 0, axis 0 1 1, limit lower=-3.14159 upper=3.14159 effort=0.0 velocity=0.0
- joint BackLeg_BackLowerLeg: axis 1 0 0 -> 0 1 0; origin xyz=0 -1 0 rpy=0 0 0 -> xyz=-1 0 0 rpy=0 0 0
- joint FrontLeg_FrontLowerLeg: axis 1 0 0 -> 0 1 0; origin xyz=0 1 0 rpy=0 0 0 -> xyz=-1 0 0 rpy=0 0 0
- joint RightLeg_RightLowerLeg: origin xyz=1 0 0 rpy=0 0 0 -> xyz=-1 0 0 rpy=0 0 0
- joint Torso_BackLeg: axis 1 0 0 -> 0 1 0; origin xyz=0 -0.5 1 rpy=0 0 0 -> xyz=-1 -0.5 1 rpy=0 0 0
- joint Torso_FrontLeg: axis 1 0 0 -> 0 1 0; origin xyz=0 0.5 1 rpy=0 0 0 -> xyz=1 0.5 1 rpy=0 0 0
- joint Torso_LeftLeg: origin xyz=-0.5 0 1 rpy=0 0 0 -> xyz=-1 0.5 1 rpy=0 0 0
- joint Torso_RightLeg: origin xyz=0.5 0 1 rpy=0 0 0 -> xyz=1 -0.5 1 rpy=0 0 0
